File: MusePad.kicad_pcb (KiCad board)
At the start: 2 copper layers, 57.4 x 44.2 mm, 26 parts, among them J1 USB_C_Receptacle_USB2.0, SW1 SW_Push, U1 ATmega32U4-AU, Y1 Crystal_GND24_Small

Commit message: gerber
Parts:
- moved F1 0.25 mm to (43.2, 98.7)
Routing:
- net VCC: track 3.75 -> 10.8 mm
- net +5V: track 119.3 -> 125.1 mm
- added copper zone on B.Cu, net GND
Changed lines of the file:
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@@
     (thickness 1.6)
     (drawings 13)
-    (tracks 292)
+    (tracks 299)
     (zones 0)
     (modules 26)
@@
   )
   (module Fuse:Fuse_1206_3216Metric (layer B.Cu)
-    (at 43.434 98.682 90)
+    (at 43.18 98.676 90)
     (descr "Fuse SMD 1206 (3216 Metric), square (rectangular) end terminal, IPC_7351 nominal, (Body size source: http://www.tortai-tech.com/upload/download/2011102023233369053.pdf), generated with kicad-footprint-generator")
     (tags resistor)
@@
   (segment (start 45.466 104.03) (end 45.596 104.16) (width 0.25) (layer B.Cu) (net 1))
   (segment (start 45.466 99.157) (end 45.466 104.03) (width 0.25) (layer B.Cu) (net 1))
-  (segment (start 44.527 94.734) (end 44.527 94.309) (width 0.25) (layer B.Cu) (net 1))
-  (segment (start 43.977 95.284) (end 44.527 94.734) (width 0.25) (layer B.Cu) (net 1))
-  (segment (start 43.552 95.284) (end 43.977 95.284) (width 0.25) (layer B.Cu) (net 1))
-  (segment (start 42.23399 96.60201) (end 43.552 95.284) (width 0.25) (layer B.Cu) (net 1))
-  (segment (start 42.23399 97.89518) (end 42.23399 96.60201) (width 0.25) (layer B.Cu) (net 1))
-  (segment (start 42.939573 98.600763) (end 42.23399 97.89518) (width 0.25) (layer B.Cu) (net 1))
-  (segment (start 44.909763 98.600763) (end 42.939573 98.600763) (width 0.25) (layer B.Cu) (net 1))
-  (segment (start 45.466 99.157) (end 44.909763 98.600763) (width 0.25) (layer B.Cu) (net 1))
   (segment (start 52.118237 98.600763) (end 51.562 99.157) (width 0.25) (layer B.Cu) (net 1))
   (segment (start 52.58701 96.34401) (end 52.58701 98.13199) (width 0.25) (layer B.Cu) (net 1))
@@
   (segment (start 91.044 102.663) (end 91.044 102.758) (width 0.25) (layer B.Cu) (net 1))
   (segment (start 91.044 102.758) (end 91.044 103.188) (width 0.25) (layer B.Cu) (net 1))
+  (segment (start 44.909763 98.600763) (end 45.466 99.157) (width 0.25) (layer B.Cu) (net 1))
+  (segment (start 42.691573 98.600763) (end 44.909763 98.600763) (width 0.25) (layer B.Cu) (net 1))
+  (segment (start 41.97999 96.66282) (end 41.97999 97.88918) (width 0.25) (layer B.Cu) (net 1))
+  (segment (start 42.31682 96.32599) (end 41.97999 96.66282) (width 0.25) (layer B.Cu) (net 1))
+  (segment (start 42.93501 96.32599) (end 42.31682 96.32599) (width 0.25) (layer B.Cu) (net 1))
+  (segment (start 44.527 94.734) (end 42.93501 96.32599) (width 0.25) (layer B.Cu) (net 1))
+  (segment (start 41.97999 97.88918) (end 42.691573 98.600763) (width 0.25) (layer B.Cu) (net 1))
+  (segment (start 44.527 94.309) (end 44.527 94.734) (width 0.25) (layer B.Cu) (net 1))
   (segment (start 81.344 114.647) (end 81.344 112.888) (width 0.25) (layer B.Cu) (net 2))
   (segment (start 79.913 116.078) (end 81.344 114.647) (width 0.25) (layer B.Cu) (net 2))
@@
   (segment (start 43.434 108.615) (end 43.337 108.712) (width 0.25) (layer B.Cu) (net 2))
   (segment (start 43.434 108.615) (end 43.434 100.082) (width 0.25) (layer B.Cu) (net 2))
+  (segment (start 82.044 106.388) (end 84.444 103.988) (width 0.25) (layer B.Cu) (net 2))
+  (segment (start 79.644 106.388) (end 82.044 106.388) (width 0.25) (layer B.Cu) (net 2))
   (segment (start 85.344 100.488) (end 85.344 101.488) (width 0.25) (layer B.Cu) (net 3))
   (segment (start 85.344 99.57) (end 85.344 100.488) (width 0.25) (layer B.Cu) (net 3))
@@
   (segment (start 45.302 95.414) (end 45.302 94.309) (width 0.25) (layer B.Cu) (net 12))
   (segment (start 43.434 97.282) (end 45.302 95.414) (width 0.25) (layer B.Cu) (net 12))
+  (segment (start 50.202 93.548998) (end 50.202 94.309) (width 0.25) (layer B.Cu) (net 12))
+  (segment (start 49.461992 92.80899) (end 50.202 93.548998) (width 0.25) (layer B.Cu) (net 12))
+  (segment (start 46.042008 92.80899) (end 49.461992 92.80899) (width 0.25) (layer B.Cu) (net 12))
+  (segment (start 45.302 94.309) (end 45.302 93.548998) (width 0.25) (layer B.Cu) (net 12))
+  (segment (start 45.302 93.548998) (end 46.042008 92.80899) (width 0.25) (layer B.Cu) (net 12))
   (segment (start 91.44 120.142) (end 96.266 120.142) (width 0.25) (layer F.Cu) (net 13))
   (segment (start 96.266 120.142) (end 96.266 108.84041) (width 0.25) (layer F.Cu) (net 13))
@@
   (segment (start 49.502 95.222) (end 49.502 94.309) (width 0.25) (layer B.Cu) (net 45))
   (segment (start 51.562 97.282) (end 49.502 95.222) (width 0.25) (layer B.Cu) (net 45))
+  (zone (net 1) (net_name GND) (layer B.Cu) (hatch edge 0.508)
+    (connect_pads (clearance 0.508))
+    (min_thickness 0.254)
+    (fill yes (arc_segments 32) (thermal_gap 0.508) (thermal_bridge_width 0.508))
+    (polygon
+      (pts
+        (xy 77.47 94.488) (xy 77.47 100.076) (xy 94.742 100.076) (xy 94.742 94.488)
+      )
+    )
+  )
 )
